File: PCB/PicoBreakout.brd (EAGLE design)
At the start: 43 parts

Commit message: PCB v2
Parts:
- moved U$3 30.8 mm to (65.1, 45.4)
Routing:
- net N$58: track 0.00 -> 113.9 mm
- net N$57: track 0.00 -> 111.0 mm, vias 1 -> 0
- net N$54: track 0.00 -> 91.4 mm
- net N$63: track 0.00 -> 88.8 mm, vias 0 -> 1
- net N$62: track 0.00 -> 75.1 mm, vias 0 -> 1
- net N$37: track 0.00 -> 42.4 mm
- net N$38: track 0.00 -> 41.9 mm
- net N$40: track 0.00 -> 40.0 mm
- net N$39: track 0.00 -> 39.8 mm
- net N$17: track 0.00 -> 24.9 mm
- net N$61: track 0.00 -> 21.8 mm, vias 0 -> 1
- net N$60: track 0.00 -> 13.3 mm, vias 0 -> 1
- net N$16: track 0.00 -> 9.92 mm
- net N$47: track 0.00 -> 5.99 mm, vias 1 -> 0
- net 14: track 92.8 -> 94.6 mm
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Other:
- board outline added: 82.5 x 57.1 mm
