File: PCB/headerboard.sch (EAGLE design)
At the start: 11 parts

Commit message: header board and schematic
Parts:
- removed T1, T2, T3, T4, T5, T6, T7, T8, T9: (no value), eagle_fab:MOSFET_NSOT23
- added 1-3, 4-6, 7-9: CONN_03_TERM'-FABLAB', fab_new:CONN_03_TERM'-FABLAB'
- added R1: (no value), fab_new:R1206FAB
- added S1: (no value), fab_new:SW_SWITCH_TACTILE_6MM6MM_SWITCH
- added U$10, U$11, U$12, U$13, U$14, U$15, U$3, U$4, U$5, U$6, U$7, U$8, U$9: SOT23NMOS, ContunityTestingRig:SOT23NMOS
- added U$2: SW_SPDTSWITCH, fab_new:SW_SPDTSWITCH
- renumbered U$1 to U$19
Connections:
- new net GND: JP1.21, S1.P, S1.P1, U$2.1
- new net N$20: 7-9.1, JP1.13, U$9.S
- new net N$21: JP1.10, U$19.P$5, U$7.D
- new net N$22: 7-9.2, JP1.15, U$10.S
- new net N$23: 7-9.3, JP1.17, U$11.S
- new net N$24: JP1.25, U$12.S
- new net N$25: JP1.27, U$13.S
- new net N$26: JP1.29, U$14.S
- new net N$27: JP1.31, U$15.S
- new net N$37: 1-3.1, JP1.1, U$3.S
- new net VCC: JP1.22, R1.2
- net N$1: now also U$10.G, U$11.G, U$12.G, U$13.G, U$14.G, U$15.G, U$2.2, U$3.G, U$4.G, U$5.G, U$6.G, U$7.G, U$8.G, U$9.G; no longer JP1.1, T1.G, T2.G, T3.G, T4.G, T5.G, T6.G, T7.G, T8.G, T9.G
- net N$10: now also JP1.18, U$11.D, U$19.P$9; no longer JP1.26, T9.D
- net N$11: now also 1-3.2, JP1.3, U$4.S; no longer JP1.19, T1.S
- net N$12: now also JP1.28, U$14.D, U$19.P$12; no longer JP1.17, T2.S
- net N$13: now also JP1.24, U$12.D, U$19.P$10; no longer JP1.15, T3.S
- net N$14: now also JP1.30, U$15.D, U$19.P$13; no longer JP1.13, T4.S
- net N$15: now also 1-3.3, JP1.5, U$5.S; no longer JP1.11, T5.S
- net N$16: now also JP1.20, R1.1, S1.S, S1.S1; no longer JP1.9, T6.S
- net N$17: now also 4-6.1, U$6.S; no longer T7.S
- net N$18: now also 4-6.2, JP1.9, U$7.S; no longer JP1.5, T8.S
- net N$19: now also 4-6.3, JP1.11, U$8.S; no longer JP1.3, T9.S
- net N$2: now also JP1.2, U$19.P$1, U$3.D; no longer JP1.6, T1.D
- net N$3: now also JP1.4, U$19.P$2, U$4.D; no longer JP1.14, T2.D
- net N$4: now also JP1.6, U$19.P$3, U$5.D; no longer JP1.8, T3.D
- net N$5: now also JP1.8, U$19.P$4, U$6.D; no longer JP1.16, T4.D
- net N$6: now also JP1.12, U$19.P$6, U$8.D; no longer JP1.10, T5.D
- net N$7: now also JP1.26, U$13.D, U$19.P$11; no longer JP1.18, T6.D
- net N$8: now also JP1.14, U$19.P$7, U$9.D; no longer JP1.12, T7.D
- net N$9: now also JP1.16, U$10.D, U$19.P$8; no longer JP1.24, T8.D

Commit message: Updates
Parts:
- added R2: 330ohm, fab_new:R1206FAB
- added U$1: LED, eagle_fab:LED
Connections:
- new net N$28: JP1.33, R2.1
- new net N$29: R2.2, U$1.A
- net GND: now also U$1.C
Changed lines of the file:
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@@
 <part name="7-9" library="fab_new" deviceset="CONN_03_TERM" device="'-FABLAB'"/>
 <part name="U$19" library="ContunityTestingRig" deviceset="13PINHEADER" device=""/>
+<part name="U$1" library="eagle_fab" deviceset="LED" device=""/>
+<part name="SUPPLY4" library="supply2" library_urn="urn:adsk.eagle:library:372" deviceset="GND" device=""/>
+<part name="R2" library="fab_new" deviceset="R" device="1206FAB" value="330ohm"/>
 </parts>
 <sheets>
@@
 </instance>
 <instance part="U$19" gate="G$1" x="78.74" y="152.4" smashed="yes"/>
+<instance part="U$1" gate="G$1" x="96.52" y="99.06" smashed="yes">
+<attribute name="NAME" x="100.076" y="97.028" size="1.778" layer="95" rot="R90"/>
+<attribute name="VALUE" x="102.235" y="97.028" size="1.778" layer="96" rot="R90"/>
+</instance>
+<instance part="SUPPLY4" gate="GND" x="96.52" y="93.98" smashed="yes">
+<attribute name="VALUE" x="94.615" y="90.805" size="1.778" layer="96"/>
+</instance>
+<instance part="R2" gate="G$1" x="86.36" y="93.98" smashed="yes">
+<attribute name="NAME" x="82.55" y="95.4786" size="1.778" layer="95"/>
+<attribute name="VALUE" x="82.55" y="90.678" size="1.778" layer="96"/>
+</instance>
 </instances>
 <busses>
@@
 <pinref part="SUPPLY3" gate="GND" pin="GND"/>
 <pinref part="U$2" gate="G$1" pin="1"/>
+</segment>
+<segment>
+<pinref part="SUPPLY4" gate="GND" pin="GND"/>
+<pinref part="U$1" gate="G$1" pin="C"/>
 </segment>
 </net>
@@
 </segment>
 </net>
+<net name="N$29" class="0">
+<segment>
+<wire x1="91.44" y1="93.98" x2="91.44" y2="104.14" width="0.1524" layer="91"/>
+<pinref part="U$1" gate="G$1" pin="A"/>
+<wire x1="91.44" y1="104.14" x2="96.52" y2="104.14" width="0.1524" layer="91"/>
+<pinref part="R2" gate="G$1" pin="2"/>
+</segment>
+</net>
+<net name="N$28" class="0">
+<segment>
+<pinref part="JP1" gate="A" pin="33"/>
+<wire x1="76.2" y1="104.14" x2="76.2" y2="93.98" width="0.1524" layer="91"/>
+<pinref part="R2" gate="G$1" pin="1"/>
+<wire x1="76.2" y1="93.98" x2="81.28" y2="93.98" width="0.1524" layer="91"/>
+</segment>
+</net>
